File: kicad_template.kicad_pcb (KiCad board)
At the start: 4 copper layers, 100 x 100 mm, 0 parts

Commit message: Update PCB template
Routing:
- added copper zone on In1.Cu, net (none)
- added copper zone on In2.Cu, net (none)
Changed lines of the file:
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@@
       (layerselection 0x00010fc_ffffffff)
       (disableapertmacros false)
-      (usegerberextensions false)
-      (usegerberattributes true)
-      (usegerberadvancedattributes true)
-      (creategerberjobfile true)
+      (usegerberextensions true)
+      (usegerberattributes false)
+      (usegerberadvancedattributes false)
+      (creategerberjobfile false)
       (svguseinch false)
       (svgprecision 6)
@@
       (plotinvisibletext false)
       (sketchpadsonfab false)
-      (subtractmaskfromsilk false)
+      (subtractmaskfromsilk true)
       (outputformat 1)
       (mirror false)
-      (drillshape 1)
+      (drillshape 0)
       (scaleselection 1)
-      (outputdirectory "")
+      (outputdirectory "gerbers")
     )
   )
@@
   (gr_line (start 101.6 50.8) (end 101.6 150.8) (layer "Edge.Cuts") (width 0.1))
   (gr_line (start 101.6 50.8) (end 201.6 50.8) (layer "Edge.Cuts") (width 0.1))
+  (zone (net 0) (net_name "") (layers "In1.Cu" "In2.Cu") (hatch edge 0.508)
+    (connect_pads (clearance 0.33))
+    (min_thickness 0.127) (filled_areas_thickness no)
+    (fill yes (thermal_gap 0.508) (thermal_bridge_width 0.508))
+    (polygon
+      (pts
+        (xy 201.6 50.8)
+        (xy 201.6 150.8)
+        (xy 101.6 150.8)
+        (xy 101.6 50.8)
+      )
+    )
+  )
 )
